File: domodisp/project/dispenc.kicad_pcb (KiCad board)
At the start: 2 copper layers, 100 x 85 mm, 29 parts, among them P1 CONN_02X05, P2 CONN_01X03, SW1 Rotary_Encoder_Switch, U1 AP111733, U2 ESP-12

Commit message: DomoDisp is now certified by OSHWA (IT000003)
Parts:
- added OSHW_Mono_0.25_Scale: IT00003, AAA mie lib verificate:OSHW_Mono_0.25_Scale, B.Cu at (150.4, 72.6)
Changed lines of the file:
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@@
-(kicad_pcb (version 4) (host pcbnew 4.0.2+dfsg1-stable)
+(kicad_pcb (version 4) (host pcbnew 4.0.5+dfsg1-4)
   (general
     (links 52)
     (no_connects 0)
-    (area 60.900001 62.299595 197.6 164.200001)
+    (area 72.924999 68.924999 173.075001 154.075001)
     (thickness 1.6)
     (drawings 32)
     (tracks 197)
     (zones 0)
-    (modules 29)
+    (modules 30)
     (nets 23)
   )
@@
     )
   )
+  (module "AAA mie lib verificate:OSHW_Mono_0.25_Scale" (layer B.Cu)
+    (at 150.368 72.644 180)
+    (fp_text reference OSHW_Mono_0.25_Scale (at 0 5.758378 180) (layer B.SilkS) hide
+      (effects (font (thickness 0.3048)) (justify mirror))
+    )
+    (fp_text value IT00003 (at 0 -4.5 180) (layer B.SilkS)
+      (effects (font (size 1.475 1.475) (thickness 0.2)) (justify mirror))
+    )
+    (fp_poly (pts (xy -5.205677 2.09181) (xy -5.205677 1.880143) (xy -5.205677 -2.498711) (xy -5.205677 -2.710378)
+      (xy -4.99401 -2.710378) (xy 4.99401 -2.710378) (xy 5.205677 -2.710378) (xy 5.205677 -2.498711)
+      (xy 5.205677 2.09181) (xy 4.791431 2.09181) (xy 4.782344 -2.287045) (xy -4.782344 -2.287045)
+      (xy -4.782344 1.668476) (xy 3.355799 1.668476) (xy 3.355799 2.09181) (xy -4.99401 2.09181)
+      (xy -5.205677 2.09181)) (layer B.SilkS) (width 0.00254))
+    (fp_poly (pts (xy -2.762961 -0.360994) (xy -2.414042 -0.360994) (xy -2.417247 -0.517108) (xy -2.426859 -0.662991)
+      (xy -2.442879 -0.798642) (xy -2.465307 -0.92406) (xy -2.494142 -1.039247) (xy -2.529385 -1.144202)
+      (xy -2.571036 -1.238925) (xy -2.619094 -1.323416) (xy -2.692866 -1.42043) (xy -2.77858 -1.499805)
+      (xy -2.876237 -1.561541) (xy -2.985837 -1.605638) (xy -3.10738 -1.632096) (xy -3.240865 -1.640916)
+      (xy -3.374351 -1.632142) (xy -3.495895 -1.605822) (xy -3.605494 -1.561954) (xy -3.703151 -1.500539)
+      (xy -3.788865 -1.421578) (xy -3.862636 -1.325069) (xy -3.910307 -1.240914) (xy -3.951623 -1.146372)
+      (xy -3.986582 -1.041444) (xy -4.015185 -0.926128) (xy -4.037431 -0.800425) (xy -4.053322 -0.664335)
+      (xy -4.062856 -0.517858) (xy -4.066034 -0.360994) (xy -4.062856 -0.204492) (xy -4.053322 -0.058274)
+      (xy -4.037431 0.07766) (xy -4.015185 0.203311) (xy -3.986582 0.318679) (xy -3.951623 0.423763)
+      (xy -3.910307 0.518564) (xy -3.862636 0.603082) (xy -3.788406 0.700095) (xy -3.702416 0.779469)
+      (xy -3.604668 0.841205) (xy -3.495159 0.885302) (xy -3.373892 0.911761) (xy -3.240865 0.920582)
+      (xy -3.10738 0.911761) (xy -2.985837 0.885302) (xy -2.876237 0.841205) (xy -2.77858 0.779469)
+      (xy -2.692866 0.700095) (xy -2.619094 0.603082) (xy -2.571036 0.518564) (xy -2.529385 0.423763)
+      (xy -2.494142 0.318679) (xy -2.465307 0.203311) (xy -2.442879 0.07766) (xy -2.426859 -0.058274)
+      (xy -2.417247 -0.204492) (xy -2.414042 -0.360994) (xy -2.762961 -0.360994) (xy -2.766085 -0.18828)
+      (xy -2.775456 -0.032838) (xy -2.791074 0.105333) (xy -2.812939 0.226233) (xy -2.841051 0.329862)
+      (xy -2.875409 0.41622) (xy -2.939799 0.518228) (xy -3.022171 0.591091) (xy -3.122527 0.63481)
+      (xy -3.240865 0.649384) (xy -3.358585 0.63481) (xy -3.458734 0.591091) (xy -3.541312 0.518228)
+      (xy -3.606321 0.41622) (xy -3.640175 0.329862) (xy -3.667874 0.226233) (xy -3.689417 0.105333)
+      (xy -3.704805 -0.032838) (xy -3.714038 -0.18828) (xy -3.717115 -0.360994) (xy -3.714038 -0.533203)
+      (xy -3.704805 -0.688232) (xy -3.689417 -0.826082) (xy -3.667874 -0.946752) (xy -3.640175 -1.050243)
+      (xy -3.606321 -1.136554) (xy -3.541312 -1.238563) (xy -3.458734 -1.311427) (xy -3.358585 -1.355145)
+      (xy -3.240865 -1.369718) (xy -3.122527 -1.355249) (xy -3.022171 -1.31184) (xy -2.939799 -1.239493)
+      (xy -2.875409 -1.138208) (xy -2.841051 -1.051851) (xy -2.812939 -0.948222) (xy -2.791074 -0.827322)
+      (xy -2.775456 -0.689151) (xy -2.766085 -0.533708) (xy -2.762961 -0.360994)) (layer B.SilkS) (width 0.00254))
+    (fp_poly (pts (xy -0.54873 0.791598) (xy -0.54873 0.4526) (xy -0.650338 0.512313) (xy -0.752313 0.561372)
+      (xy -0.854654 0.599775) (xy -0.956446 0.627334) (xy -1.058972 0.64387) (xy -1.162232 0.649384)
+      (xy -1.308856 0.637072) (xy -1.433431 0.60014) (xy -1.535956 0.53859) (xy -1.612208 0.457192)
+      (xy -1.657959 0.358525) (xy -1.673209 0.242587) (xy -1.650885 0.098305) (xy -1.583912 -0.007114)
+      (xy -1.506007 -0.061318) (xy -1.393559 -0.109273) (xy -1.246568 -0.150981) (xy -1.071282 -0.190668)
+      (xy -0.939917 -0.226784) (xy -0.823633 -0.270309) (xy -0.72243 -0.321241) (xy -0.636307 -0.379581)
+      (xy -0.565266 -0.445329) (xy -0.495814 -0.540001) (xy -0.446205 -0.650382) (xy -0.416439 -0.776473)
+      (xy -0.406516 -0.918272) (xy -0.415248 -1.052482) (xy -0.441442 -1.173331) (xy -0.485098 -1.280818)
+      (xy -0.546217 -1.374943) (xy -0.624797 -1.455708) (xy -0.720048 -1.522383) (xy -0.831173 -1.574241)
+      (xy -0.958173 -1.611283) (xy -1.101048 -1.633508) (xy -1.259797 -1.640916) (xy -1.375737 -1.63669)
+      (xy -1.492043 -1.624012) (xy -1.608717 -1.602881) (xy -1.725758 -1.574402) (xy -1.843167 -1.537471)
+      (xy -1.960943 -1.492087) (xy -1.960943 -1.136554) (xy -1.836552 -1.209866) (xy -1.716939 -1.268846)
+      (xy -1.602102 -1.313494) (xy -1.488368 -1.34473) (xy -1.374267 -1.363471) (xy -1.259797 -1.369718)
+      (xy -1.140322 -1.36269) (xy -1.034902 -1.341606) (xy -0.943538 -1.306466) (xy -0.86623 -1.25727)
+      (xy -0.788142 -1.171281) (xy -0.741288 -1.065447) (xy -0.72567 -0.93977) (xy -0.736511 -0.826036)
+      (xy -0.769033 -0.731778) (xy -0.823234 -0.656996) (xy -0.903162 -0.596914) (xy -1.015059 -0.546754)
+      (xy -1.158925 -0.506514) (xy -1.337519 -0.465173) (xy -1.467562 -0.43091) (xy -1.582523 -0.390297)
+      (xy -1.682403 -0.343334) (xy -1.767202 -0.29002) (xy -1.83692 -0.230356) (xy -1.904926 -0.145091)
+      (xy -1.953502 -0.046389) (xy -1.982647 0.065749) (xy -1.992363 0.191324) (xy -1.983499 0.318323)
+      (xy -1.956909 0.434739) (xy -1.912591 0.540572) (xy -1.850546 0.635823) (xy -1.770774 0.72049)
+      (xy -1.675656 0.792522) (xy -1.568897 0.848547) (xy -1.450496 0.888565) (xy -1.320453 0.912577)
+      (xy -1.178769 0.920582) (xy -1.082307 0.916905) (xy -0.982537 0.905881) (xy -0.879459 0.887509)
+      (xy -0.772892 0.862886) (xy -0.662649 0.830916) (xy -0.54873 0.791598)) (layer B.SilkS) (width 0.00254))
+    (fp_poly (pts (xy 0.041622 0.875933) (xy 0.377312 0.875933) (xy 0.377312 -0.136098) (xy 1.291778 -0.136098)
+      (xy 1.291778 0.875933) (xy 1.627468 0.875933) (xy 1.627468 -1.59296) (xy 1.291778 -1.59296)
+      (xy 1.291778 -0.417218) (xy 0.377312 -0.417218) (xy 0.377312 -1.59296) (xy 0.041622 -1.59296)
+      (xy 0.041622 0.875933)) (layer B.SilkS) (width 0.00254))
+    (fp_poly (pts (xy 1.852364 0.875933) (xy 2.178133 0.875933) (xy 2.414604 -1.128285) (xy 2.695723 0.197938)
+      (xy 3.044643 0.197938) (xy 3.32907 -1.131593) (xy 4.129986 2.710378) (xy 4.455754 2.710378)
+      (xy 3.522546 -1.59296) (xy 3.2067 -1.59296) (xy 2.87101 -0.126176) (xy 2.536973 -1.59296)
+      (xy 2.221127 -1.59296) (xy 1.852364 0.875933)) (layer B.SilkS) (width 0.00254))
+  )
   (dimension 25 (width 0.3) (layer Dwgs.User)
