File: domonode-inout/project/domonode-inout.sch (KiCad schematic (older format))
At the start: 51 parts, among them P1 CONN_01X03, P10 CONN_01X02, P11 CONN_01X02, P12 CONN_01X02, P13 CONN_01X02, P2 CONN_2x5, P3 CONN_01X03, P4 CONN_01X03, P5 CONN_01X03, P6 CONN_01X02, P7 CONN_01X02, P8 CONN_01X02, P9 CONN_01X02, U1 HLK-PM01, U2 PCA9555, U3 TLP620, U4 TLP620, U5 TLP620, U6 24LC02

Commit message: Updated DomoNode-Inout to 1.1.2 (improved connectors footprints)
Parts:
- removed P1, P3, P4, P5: CONN_01X03, Connect:AK300-3, symbol CONN_01X03
- added P1, P3, P4, P5: CONN_01X02, AAA mie lib verificate:KF2EDGK-5.08-2, symbol CONN_01X02
- added P2: Conn_01x04, AAA mie lib verificate:KF2EDGK-5.08-4, symbol Conn_01x04
- C4, C6, C8: footprint Capacitors_ThroughHole:C_Rect_L18.0mm_W6.0mm_P15.00mm_FKS3_FKP3 -> Capacitors_ThroughHole:C_Rect_L13.0mm_W6.0mm_P10.00mm_FKS3_FKP3_MKS4
- renumbered P2 to J1
Connections:
- net I1L: now also P3.1 (P1)
- net I1N: now also P3.2 (P2)
- net I2L: now also P4.1 (P1)
- net I2N: now also P4.2 (P2)
- net I3L: now also P5.1 (P1)
- net I3N: now also P5.2 (P2)
- net L: now also P1.1 (P1)
- net N: now also P1.2 (P2)
- net RL1P: now also P2.1 (Pin_1)
- net RL2P: now also P2.2 (Pin_2)
- net RL3P: now also P2.3 (Pin_3)
- net RL4P: now also P2.4 (Pin_4)
Other:
- note added: "Note: if only one expansion module is needed, avoid mounting power section and close J4.\nAt power on IOx lines are INPUTS pulled HIGH via weak pull-ups.\n"
- note removed: "Note: Omron G3MB-202 (2A SSR) can be replaced by Panasonic APAN3105 (5A relays)\nIf only one expansion module is needed, avoid mounting power section and close J4.\nIOx lines are HIGH at power on via pull-ups.\n"
Changed lines of the file:
@@
 LIBS:ssr
 LIBS:power
-LIBS:device
-LIBS:transistors
 LIBS:conn
-LIBS:linear
-LIBS:regul
-LIBS:74xx
-LIBS:cmos4000
-LIBS:adc-dac
-LIBS:memory
-LIBS:xilinx
-LIBS:microcontrollers
-LIBS:dsp
-LIBS:microchip
-LIBS:analog_switches
-LIBS:motorola
-LIBS:texas
-LIBS:intel
-LIBS:audio
-LIBS:interface
-LIBS:digital-audio
-LIBS:philips
-LIBS:display
-LIBS:cypress
-LIBS:siliconi
-LIBS:opto
-LIBS:atmel
-LIBS:contrib
-LIBS:valves
-LIBS:switches
-LIBS:pca9555
 LIBS:domonode-inout-cache
 EELAYER 25 0
@@
 Sheet 1 1
 Title "DomoNode-inout"
-Date "2018-01-08"
-Rev "1.1.1"
+Date "2018-05-13"
+Rev "1.1.2"
 Comp "CSSHL.org"
 Comment1 ""
@@
 $EndComp
 $Comp
-L CONN_01X03 P1
-U 1 1 5989A97A
-P 1000 2700
-F 0 "P1" H 1000 2900 50  0000 C CNN
-F 1 "CONN_01X03" V 1100 2700 50  0000 C CNN
-F 2 "Connect:AK300-3" H 1000 2700 50  0001 C CNN
-F 3 "" H 1000 2700 50  0000 C CNN
-	1    1000 2700
-	-1   0    0    -1
-$EndComp
-$Comp
-L CONN_01X10 P2
+L CONN_01X10 J1
 U 1 1 598D80AA
 P 10450 4400
-F 0 "P2" H 10450 4900 50  0000 C CNN
+F 0 "J1" H 10450 4950 50  0000 C CNN
 F 1 "CONN_2x5" V 10550 4400 50  0001 C CNN
 F 2 "Connectors_Multicomp:Multicomp_MC9A12-1034_2x05x2.54mm_Straight" V 10450 4400 50  0001 C CNN
@@
 	1    2400 2550
 	1    0    0    -1
-$EndComp
-$Comp
-L CONN_01X03 P3
-U 1 1 598F3421
-P 1000 3200
-F 0 "P3" H 1000 3400 50  0000 C CNN
-F 1 "CONN_01X03" V 1100 3200 50  0000 C CNN
-F 2 "Connect:AK300-3" H 1000 3200 50  0001 C CNN
-F 3 "" H 1000 3200 50  0000 C CNN
-	1    1000 3200
-	-1   0    0    -1
 $EndComp
 Wire Wire Line
@@
 Wire Wire Line
 	2450 1700 2100 1700
-Text Notes 7050 7100 0    60   ~ 0
-Note: Omron G3MB-202 (2A SSR) can be replaced by Panasonic APAN3105 (5A relays)\nIf only one expansion module is needed, avoid mounting power section and close J4.\nIOx lines are HIGH at power on via pull-ups.\n
+Text Notes 7000 7000 0    60   ~ 0
+Note: if only one expansion module is needed, avoid mounting power section and close J4.\nAt power on IOx lines are INPUTS pulled HIGH via weak pull-ups.\n
 Wire Wire Line
 	1800 1700 1600 1700
@@
 Text Label 1700 2950 2    60   ~ 0
 RL2P
-Text Label 1200 2800 0    60   ~ 0
+Text Label 1200 3000 0    60   ~ 0
 RL1P
 Text Label 1200 3100 0    60   ~ 0
@@
 Wire Wire Line
 	10250 2000 10450 2000
-$Comp
-L CONN_01X03 P4
-U 1 1 59EDBBC5
-P 1000 3700
-F 0 "P4" H 1000 3900 50  0000 C CNN
-F 1 "CONN_01X03" V 1100 3700 50  0000 C CNN
-F 2 "Connect:AK300-3" H 1000 3700 50  0001 C CNN
-F 3 "" H 1000 3700 50  0000 C CNN
-	1    1000 3700
-	-1   0    0    -1
-$EndComp
-$Comp
-L CONN_01X03 P5
-U 1 1 59EDD1CF
-P 1000 4200
-F 0 "P5" H 1000 4400 50  0000 C CNN
-F 1 "CONN_01X03" V 1100 4200 50  0000 C CNN
-F 2 "Connect:AK300-3" H 1000 4200 50  0001 C CNN
-F 3 "" H 1000 4200 50  0000 C CNN
-	1    1000 4200
-	-1   0    0    -1
-$EndComp
 Text Label 1200 3600 0    60   ~ 0
 I1L
 Text Label 1200 3700 0    60   ~ 0
 I1N
-Text Label 1200 3800 0    60   ~ 0
+Text Label 1200 3950 0    60   ~ 0
 I2L
-Text Label 1200 4100 0    60   ~ 0
+Text Label 1200 4050 0    60   ~ 0
 I2N
-Text Label 1200 4200 0    60   ~ 0
+Text Label 1200 4300 0    60   ~ 0
 I3L
-Text Label 1200 4300 0    60   ~ 0
+Text Label 1200 4400 0    60   ~ 0
 I3N
 Text Label 4250 3700 2    60   ~ 0
@@
 F 0 "C4" H 4425 3000 50  0000 L CNN
 F 1 "0.1uF X2" H 4425 2800 50  0000 L CNN
-F 2 "Capacitors_ThroughHole:C_Rect_L18.0mm_W6.0mm_P15.00mm_FKS3_FKP3" H 4438 2750 50  0001 C CNN
+F 2 "Capacitors_ThroughHole:C_Rect_L13.0mm_W6.0mm_P10.00mm_FKS3_FKP3_MKS4" H 4438 2750 50  0001 C CNN
 F 3 "" H 4400 2900 50  0000 C CNN
 	1    4400 2900
@@
 F 0 "C6" H 4425 4000 50  0000 L CNN
 F 1 "0.1uF X2" H 4425 3800 50  0000 L CNN
-F 2 "Capacitors_ThroughHole:C_Rect_L18.0mm_W6.0mm_P15.00mm_FKS3_FKP3" H 4438 3750 50  0001 C CNN
+F 2 "Capacitors_ThroughHole:C_Rect_L13.0mm_W6.0mm_P10.00mm_FKS3_FKP3_MKS4" H 4438 3750 50  0001 C CNN
 F 3 "" H 4400 3900 50  0000 C CNN
 	1    4400 3900
@@
 F 0 "C8" H 4425 5000 50  0000 L CNN
 F 1 "0.1uF X2" H 4425 4800 50  0000 L CNN
-F 2 "Capacitors_ThroughHole:C_Rect_L18.0mm_W6.0mm_P15.00mm_FKS3_FKP3" H 4438 4750 50  0001 C CNN
+F 2 "Capacitors_ThroughHole:C_Rect_L13.0mm_W6.0mm_P10.00mm_FKS3_FKP3_MKS4" H 4438 4750 50  0001 C CNN
 F 3 "" H 4400 4900 50  0000 C CNN
 	1    4400 4900
@@
 	1    0    0    -1
 $EndComp
+$Comp
+L CONN_01X02 P3
+U 1 1 5AF87CAC
+P 1000 3650
+F 0 "P3" H 1000 3800 50  0000 C CNN
+F 1 "CONN_01X02" V 1100 3650 50  0000 C CNN
+F 2 "AAA mie lib verificate:KF2EDGK-5.08-2" H 1000 3650 50  0001 C CNN
+F 3 "" H 1000 3650 50  0000 C CNN
+	1    1000 3650
+	-1   0    0    -1
+$EndComp
+$Comp
+L CONN_01X02 P4
+U 1 1 5AF87D9A
+P 1000 4000
+F 0 "P4" H 1000 4150 50  0000 C CNN
+F 1 "CONN_01X02" V 1100 4000 50  0000 C CNN
+F 2 "AAA mie lib verificate:KF2EDGK-5.08-2" H 1000 4000 50  0001 C CNN
+F 3 "" H 1000 4000 50  0000 C CNN
+	1    1000 4000
+	-1   0    0    -1
+$EndComp
+$Comp
+L CONN_01X02 P5
+U 1 1 5AF87E79
+P 1000 4350
+F 0 "P5" H 1000 4500 50  0000 C CNN
+F 1 "CONN_01X02" V 1100 4350 50  0000 C CNN
+F 2 "AAA mie lib verificate:KF2EDGK-5.08-2" H 1000 4350 50  0001 C CNN
+F 3 "" H 1000 4350 50  0000 C CNN
+	1    1000 4350
+	-1   0    0    -1
+$EndComp
+$Comp
+L Conn_01x04 P2
+U 1 1 5AF882DC
+P 1000 3100
+F 0 "P2" H 1000 3300 50  0000 C CNN
+F 1 "Conn_01x04" V 1100 3050 50  0000 C CNN
+F 2 "AAA mie lib verificate:KF2EDGK-5.08-4" H 1000 3100 50  0001 C CNN
+F 3 "" H 1000 3100 50  0001 C CNN
+	1    1000 3100
+	-1   0    0    -1
+$EndComp
+$Comp
+L CONN_01X02 P1
+U 1 1 5AF8843D
+P 1000 2650
+F 0 "P1" H 1000 2800 50  0000 C CNN
+F 1 "CONN_01X02" V 1100 2650 50  0000 C CNN
+F 2 "AAA mie lib verificate:KF2EDGK-5.08-2" H 1000 2650 50  0001 C CNN
+F 3 "" H 1000 2650 50  0000 C CNN
+	1    1000 2650
+	-1   0    0    -1
+$EndComp
 $EndSCHEMATC

Commit message: DomoNode-Inout: Fixed a really stupid error (swapped SCA/SCL on PCA9555); changed connector layout in schematic (from 1x10 to 2x5) for better readability
Parts:
- J1: symbol CONN_01X10 -> Conn_02x05_Odd_Even
Connections:
- net SCL: now also R2.2, U2.22 (SCL); no longer R1.2, U2.23 (SDA)
- net SDA: now also R1.2, U2.23 (SDA); no longer R2.2, U2.22 (SCL)
Changed lines of the file:
@@
 Title "DomoNode-inout"
 Date "2018-05-13"
-Rev "1.1.2"
+Rev "1.1.3"
 Comp "CSSHL.org"
 Comment1 ""
@@
 L GND #PWR03
 U 1 1 59898E1E
-P 9900 4750
-F 0 "#PWR03" H 9900 4500 50  0001 C CNN
-F 1 "GND" H 9900 4600 50  0000 C CNN
-F 2 "" H 9900 4750 50  0000 C CNN
-F 3 "" H 9900 4750 50  0000 C CNN
-	1    9900 4750
+P 9550 4650
+F 0 "#PWR03" H 9550 4400 50  0001 C CNN
+F 1 "GND" H 9550 4500 50  0000 C CNN
+F 2 "" H 9550 4650 50  0000 C CNN
+F 3 "" H 9550 4650 50  0000 C CNN
+	1    9550 4650
 	1    0    0    -1
 $EndComp
@@
 $EndComp
 $Comp
-L CONN_01X10 J1
+L Conn_02x05_Odd_Even J1
 U 1 1 598D80AA
-P 10450 4400
-F 0 "J1" H 10450 4950 50  0000 C CNN
-F 1 "CONN_2x5" V 10550 4400 50  0001 C CNN
-F 2 "Connectors_Multicomp:Multicomp_MC9A12-1034_2x05x2.54mm_Straight" V 10450 4400 50  0001 C CNN
-F 3 "" H 10450 4400 50  0000 C CNN
-	1    10450 4400
+P 10100 4450
+F 0 "J1" H 10150 4750 50  0000 C CNN
+F 1 "CONN_2x5" V 10200 4450 50  0001 C CNN
+F 2 "Connectors_Multicomp:Multicomp_MC9A12-1034_2x05x2.54mm_Straight" V 10100 4450 50  0001 C CNN
+F 3 "" H 10100 4450 50  0000 C CNN
+	1    10100 4450
 	1    0    0    -1
 $EndComp
@@
 	4250 1600 4250 1650
 Wire Wire Line
-	9900 4750 10250 4750
+	9550 4650 9900 4650
 $Comp
 L Omron_G3MB-202 RL1
@@
 	1    0    0    -1
 $EndComp
+Text Label 9850 1800 0    60   ~ 0
+SCL
 Text Label 9850 1700 0    60   ~ 0
+SDA
+Text Label 9900 4350 2    60   ~ 0
+TXD
+Text Label 9900 4450 2    60   ~ 0
+RXD
+Text Label 10400 4450 0    60   ~ 0
+SDA
+Text Label 10400 4350 0    60   ~ 0
 SCL
-Text Label 9850 1800 0    60   ~ 0
-SDA
-Text Label 10250 4150 2    60   ~ 0
-TXD
-Text Label 10250 4350 2    60   ~ 0
-RXD
-Text Label 10250 4450 2    60   ~ 0
-SDA
-Text Label 10250 4250 2    60   ~ 0
-SCL
-Text Label 10250 4550 2    60   ~ 0
+Text Label 9900 4550 2    60   ~ 0
 PROG
-Text Label 10250 4050 2    60   ~ 0
+Text Label 10400 4250 0    60   ~ 0
 DBG
-Text Label 10250 4650 2    60   ~ 0
+Text Label 10400 4550 0    60   ~ 0
 ADC
 Text Label 7500 1700 2    60   ~ 0
@@
 L +3.3V #PWR011
 U 1 1 59E7D16B
-P 10250 3950
-F 0 "#PWR011" H 10250 3800 50  0001 C CNN
-F 1 "+3.3V" H 10250 4090 50  0000 C CNN
-F 2 "" H 10250 3950 50  0000 C CNN
-F 3 "" H 10250 3950 50  0000 C CNN
-	1    10250 3950
+P 9900 4250
+F 0 "#PWR011" H 9900 4100 50  0001 C CNN
+F 1 "+3.3V" H 9900 4390 50  0000 C CNN
+F 2 "" H 9900 4250 50  0000 C CNN
+F 3 "" H 9900 4250 50  0000 C CNN
+	1    9900 4250
 	1    0    0    -1
 $EndComp
@@
 Wire Wire Line
 	8800 2000 10050 2000
-Text Label 10250 4850 2    60   ~ 0
+Text Label 10400 4650 0    60   ~ 0
 5VEXT
 Text Label 9850 2300 2    60   ~ 0
